Commit message: fix,adjust files to my own repostory

File: description/robot_base.xacro (robot description, xacro)
@@ -146,33 +146,33 @@
         <mu2 value="0.01" />
     </gazebo>
-        <!-- RIGHT CASTER WHEELS LINK-->
-        <joint name="right_caster_wheel_joint" type="fixed">
-            <parent link="chassis" />
-            <child link="right_caster_wheel" />
-            <origin xyz="0.4 -0.175 0" rpy="${pi/2} 0 0"/>
-            <axis xyz="0 0 -1"/>
-        </joint>
-        <link name="right_caster_wheel">
-            <visual>
-                <geometry>
-                    <cylinder radius="0.05" length="0.04"/>
-                </geometry>
-                <material name="black" />
-            </visual>
-            <collision>
-                <geometry>
-                    <cylinder radius="0.05" length="0.04"/>
-                </geometry>
-            </collision>
-            <xacro:inertial_cylinder mass="0.1" length="0.04" radius="0.05">
-                <origin xyz="0 0 0" rpy="0 0 0"/>
-            </xacro:inertial_cylinder>
-        </link>
-        <gazebo reference="right_caster_wheel">
-            <material>
-                Gazebo/Black
-            </material>
-            <mu1 value="0.01" />
-            <mu2 value="0.01" />
-        </gazebo>
+    <!-- RIGHT CASTER WHEELS LINK-->
+    <joint name="right_caster_wheel_joint" type="fixed">
+        <parent link="chassis" />
+        <child link="right_caster_wheel" />
+        <origin xyz="0.4 -0.175 0" rpy="${pi/2} 0 0"/>
+        <axis xyz="0 0 -1"/>
+    </joint>
+    <link name="right_caster_wheel">
+        <visual>
+            <geometry>
+                <cylinder radius="0.05" length="0.04"/>
+            </geometry>
+            <material name="black" />
+        </visual>
+        <collision>
+            <geometry>
+                <cylinder radius="0.05" length="0.04"/>
+            </geometry>
+        </collision>
+        <xacro:inertial_cylinder mass="0.1" length="0.04" radius="0.05">
+            <origin xyz="0 0 0" rpy="0 0 0"/>
+        </xacro:inertial_cylinder>
+    </link>
+    <gazebo reference="right_caster_wheel">
+        <material>
+            Gazebo/Black
+        </material>
+        <mu1 value="0.01" />
+        <mu2 value="0.01" />
+    </gazebo>
 </robot>
